File: kicad_project/iotboard/iotboard/iotboard.sch (KiCad schematic (older format))
At the start: 0 parts

Commit message: added datasheets and project
Parts:
- added C? (x2): 10u, symbol Device:CP
- added C?: 100n, symbol Device:C
- added C? (x2): 1u, symbol Device:C
- added C? (x2): 10u, symbol Device:C
- added C?: 4.7u, symbol Device:CP
- added D? (x2): LED, symbol Device:LED
- added D?: D_Schottky, symbol Device:D_Schottky
- added J?: USB_B_Micro, symbol Connector:USB_B_Micro
- added J?: Conn_01x02, symbol Connector_Generic:Conn_01x02
- added R? (x6): 10k, symbol Device:R
- added R? (x3): 1k, symbol Device:R
- added R?: 2k, symbol Device:R
- added SW?: SW_Push, symbol Switch:SW_Push
- added U?: ESP-12F, symbol ESP8266:ESP-12F
- added U?: CP2102N-A01-GQFN24, Package_DFN_QFN:QFN-24-1EP_4x4mm_P0.5mm_EP2.6x2.6mm, symbol Interface_USB:CP2102N-A01-GQFN24
- added U?: AP2127K-3.3, Package_TO_SOT_SMD:SOT-23-5, symbol Regulator_Linear:AP2127K-3.3
- added U?: MCP73831-2-OT, Package_TO_SOT_SMD:SOT-23-5, symbol Battery_Management:MCP73831-2-OT
Connections:
- net labels added: +3.3V, +BATT, ADC0, DSR, DTR, EN, GND, GPIO0, GPIO12_MISO, GPIO13_MOSI, GPIO14_SCK, GPIO15, GPIO16, GPIO2, GPIO3, GPIO4_SDA, GPIO5_SCL, RST, RXD, STAT, TXD, VBUS
- wire segments 0 -> 136
- no-connect marks 0 -> 18
Other:
- note added: "ESP8266 Module"
- note added: "LED"
- note added: "Power"
- note added: "Reset"
- note added: "USB to serial converter"

Commit message: added the PCB layout, some libraries
Parts:
- removed C?: 4.7u, symbol Device:CP
- removed C?: 10u, symbol Device:CP
- added C5: 4.7u, Capacitors_SMD:C_0603_HandSoldering, symbol Device:C
- added C6: 10u, Capacitors_SMD:C_0603_HandSoldering, symbol Device:C
- added C7: 100n, Capacitors_SMD:C_0603_HandSoldering, symbol Device:C
- added J3: Conn_01x12, Socket_Strips:Socket_Strip_Straight_1x12_Pitch2.54mm, symbol Connector_Generic:Conn_01x12
- added J4: Conn_01x16, Socket_Strips:Socket_Strip_Straight_1x16_Pitch2.54mm, symbol Connector_Generic:Conn_01x16
- added MH1, MH2, MH3, MH4: MountingHole_Pad, Mounting_Holes:MountingHole_3mm_Pad_Via, symbol Mechanical:MountingHole_Pad
- added Q1, Q2: mmbt2222, TO_SOT_Packages_SMD:SOT-23, symbol Device:Q_NPN_BCE
- added R3, R4, R8: 10k, Resistors_SMD:R_0603_HandSoldering, symbol Device:R
- added R7: 4k7, Resistors_SMD:R_0603_HandSoldering, symbol Device:R
- added SW1: SW_Push, Buttons_Switches_SMD:SW_SPST_EVPBF, symbol Switch:SW_Push
- added U4: DHT11, Sensor:Aosong_DHT11_5.5x12.0_P2.54mm, symbol Sensor:DHT11
- C1, C2, C3, C4, C8, C9: renamed from C?; footprint (none) -> Capacitors_SMD:C_0603_HandSoldering
- D1: renamed from D?; footprint (none) -> Diodes_SMD:D_0603
- D2, D3: renamed from D?; footprint (none) -> LEDs:LED_0805_HandSoldering
- J1: renamed from J?; footprint (none) -> Connectors_JST:JST_XH_S02B-XH-A_02x2.50mm_Angled
- J2: renamed from J?; footprint (none) -> Connectors_USB:USB_Micro-B_Molex_47346-0001
- R1, R10, R11, R12, R13, R14, R2, R5, R6, R9: renamed from R?; footprint (none) -> Resistors_SMD:R_0603_HandSoldering
- SW2: renamed from SW?; footprint (none) -> Buttons_Switches_SMD:SW_SPST_EVPBF
- U1, U3: renamed from U?; footprint Package_TO_SOT_SMD:SOT-23-5 -> TO_SOT_Packages_SMD:SOT-23-5_HandSoldering
- U2: renamed from U?; footprint Package_DFN_QFN:QFN-24-1EP_4x4mm_P0.5mm_EP2.6x2.6mm -> Housings_DFN_QFN:QFN-24-1EP_4x4mm_Pitch0.5mm
- U5: renamed from U?; footprint (none) -> ESP8266:ESP-12E
Connections:
- net labels added: EN_R, RTS
- net labels removed: DSR, GPIO3
- wire segments 136 -> 210
- no-connect marks 18 -> 24
Other:
- note added: "Charger"
- note added: "Pinout"
- note added: "Push button"
- note added: "Temperature and humity sensor"
- moved on the sheet: U1, U3

Commit message: added KiCAD PCB y project
Parts:
- MH1, MH2, MH3, MH4: footprint Mounting_Holes:MountingHole_3mm_Pad_Via -> Mounting_Holes:MountingHole_2.5mm_Pad_Via
- SW1, SW2: footprint Buttons_Switches_SMD:SW_SPST_EVPBF -> Buttons_Switches_SMD:SW_SPST_PTS645
Changed lines of the file:
@@
 F 0 "SW2" V 4896 7227 50  0000 R CNN
 F 1 "SW_Push" V 4805 7227 50  0000 R CNN
-F 2 "Buttons_Switches_SMD:SW_SPST_EVPBF" H 4850 7475 50  0001 C CNN
+F 2 "Buttons_Switches_SMD:SW_SPST_PTS645" H 4850 7475 50  0001 C CNN
 F 3 "" H 4850 7475 50  0001 C CNN
 	1    4850 7275
@@
 F 0 "SW1" V 7146 5177 50  0000 R CNN
 F 1 "SW_Push" V 7055 5177 50  0000 R CNN
-F 2 "Buttons_Switches_SMD:SW_SPST_EVPBF" H 7100 5425 50  0001 C CNN
+F 2 "Buttons_Switches_SMD:SW_SPST_PTS645" H 7100 5425 50  0001 C CNN
 F 3 "" H 7100 5425 50  0001 C CNN
 	1    7100 5225
@@
 F 0 "MH3" H 7550 6101 50  0000 L CNN
 F 1 "MountingHole_Pad" H 7125 6250 50  0001 L CNN
-F 2 "Mounting_Holes:MountingHole_3mm_Pad_Via" H 7450 6050 50  0001 C CNN
+F 2 "Mounting_Holes:MountingHole_2.5mm_Pad_Via" H 7450 6050 50  0001 C CNN
 F 3 "~" H 7450 6050 50  0001 C CNN
 	1    7450 6050
@@
 F 0 "MH4" H 8000 6101 50  0000 L CNN
 F 1 "MountingHole_Pad" H 7575 6250 50  0001 L CNN
-F 2 "Mounting_Holes:MountingHole_3mm_Pad_Via" H 7900 6050 50  0001 C CNN
+F 2 "Mounting_Holes:MountingHole_2.5mm_Pad_Via" H 7900 6050 50  0001 C CNN
 F 3 "~" H 7900 6050 50  0001 C CNN
 	1    7900 6050
@@
 F 0 "MH1" H 6700 6101 50  0000 L CNN
 F 1 "MountingHole_Pad" H 6275 6250 50  0001 L CNN
-F 2 "Mounting_Holes:MountingHole_3mm_Pad_Via" H 6600 6050 50  0001 C CNN
+F 2 "Mounting_Holes:MountingHole_2.5mm_Pad_Via" H 6600 6050 50  0001 C CNN
 F 3 "~" H 6600 6050 50  0001 C CNN
 	1    6600 6050
@@
 F 0 "MH2" H 7150 6101 50  0000 L CNN
 F 1 "MountingHole_Pad" H 6725 6250 50  0001 L CNN
-F 2 "Mounting_Holes:MountingHole_3mm_Pad_Via" H 7050 6050 50  0001 C CNN
+F 2 "Mounting_Holes:MountingHole_2.5mm_Pad_Via" H 7050 6050 50  0001 C CNN
 F 3 "~" H 7050 6050 50  0001 C CNN
 	1    7050 6050
